File: Hardware/rpismdoven/_saved_rpismdoven.sch (KiCad schematic (older format))
At the start: 19 parts, among them J1 Raspberry_Pi_2_3, J2 Conn_01x02_Female, J3 T-PROBE, J4 MAX31855-BREAKOUT, Q1 2N2219, Q2 2N2219, U1 MAX31855TASA

Commit message: bump HW
Parts:
- BZ1: footprint (none) -> Buzzer_Beeper:Buzzer_15x7.5RM7.6
- Q1, Q2: footprint Package_TO_SOT_THT:TO-39-3 -> Package_TO_SOT_THT:TO-92
Changed lines of the file:
@@
 F 0 "Q2" H 4791 6346 50  0000 L CNN
 F 1 "2N2219" H 4791 6255 50  0000 L CNN
-F 2 "Package_TO_SOT_THT:TO-39-3" H 4800 6225 50  0001 L CIN
+F 2 "Package_TO_SOT_THT:TO-92" H 4800 6225 50  0001 L CIN
 F 3 "http://www.onsemi.com/pub_link/Collateral/2N2219-D.PDF" H 4600 6300 50  0001 L CNN
 	1    4600 6300
@@
 F 0 "BZ1" H 2953 5029 50  0000 L CNN
 F 1 "Buzzer" H 2953 4938 50  0000 L CNN
-F 2 "" V 2775 5100 50  0001 C CNN
+F 2 "Buzzer_Beeper:Buzzer_15x7.5RM7.6" V 2775 5100 50  0001 C CNN
 F 3 "~" V 2775 5100 50  0001 C CNN
 	1    2800 5000
@@
 F 0 "Q1" H 2716 5571 50  0000 L CNN
 F 1 "2N2219" H 2716 5480 50  0000 L CNN
-F 2 "Package_TO_SOT_THT:TO-39-3" H 2725 5450 50  0001 L CIN
+F 2 "Package_TO_SOT_THT:TO-92" H 2725 5450 50  0001 L CIN
 F 3 "http://www.onsemi.com/pub_link/Collateral/2N2219-D.PDF" H 2525 5525 50  0001 L CNN
 	1    2525 5525
