File: Hardware/rpismdoven/rpismdoven.kicad_pcb (KiCad board)
At the start: 2 copper layers, 2 parts

Commit message: bump HW
Parts:
- removed the REF** at (128.9, 73.7)
- added BZ1: Buzzer, Buzzer_Beeper:Buzzer_15x7.5RM7.6, F.Cu at (106.3, 97.2)
- added C1: 10nF, Capacitor_SMD:C_0603_1608Metric, F.Cu at (119.0, 75.5)
- added C2: 10uF, Capacitor_SMD:C_0603_1608Metric, F.Cu at (154.4, 84.9)
- added C3: 10uF, Capacitor_SMD:C_0603_1608Metric, F.Cu at (115.3, 73.3)
- added D1: 1N4148, Diode_THT:D_DO-35_SOD27_P7.62mm_Horizontal, F.Cu at (128.9, 96.0)
- added D2: 1N4148, Diode_THT:D_DO-35_SOD27_P7.62mm_Horizontal, F.Cu at (131.9, 88.4)
- added J1: Raspberry_Pi_2_3, Connector_PinSocket_2.54mm:PinSocket_2x20_P2.54mm_Vertical, B.Cu at (107.1, 60.2)
- added J2: Conn_01x02_Female, TerminalBlock:TerminalBlock_bornier-2_P5.08mm, F.Cu at (102.9, 66.3)
- added J3: T-PROBE, TerminalBlock:TerminalBlock_bornier-2_P5.08mm, F.Cu at (134.3, 71.2)
- added J4: MAX31855-BREAKOUT, Connector_PinSocket_2.54mm:PinSocket_1x06_P2.54mm_Vertical, F.Cu at (120.2, 89.2)
- added L1: Ferrite_Bead_Small, Inductor_SMD:L_0603_1608Metric, F.Cu at (136.8, 78.2)
- added L2: Ferrite_Bead_Small, Inductor_SMD:L_0603_1608Metric, F.Cu at (133.4, 78.1)
- added Q1: 2N2219, Package_TO_SOT_THT:TO-92, F.Cu at (149.5, 101.5)
- added Q2: 2N2219, Package_TO_SOT_THT:TO-92, F.Cu at (148.0, 89.8)
- added R1: 1k, Resistor_SMD:R_0603_1608Metric, F.Cu at (144.5, 82.7)
- added R2: 1k, Resistor_SMD:R_0603_1608Metric, F.Cu at (148.9, 77.9)
- added R3: R_Small, Resistor_SMD:R_0603_1608Metric, F.Cu at (127.7, 100.7)
- added R4: R_Small, Resistor_SMD:R_0603_1608Metric, F.Cu at (131.5, 100.5)
- added U1: MAX31855TASA, Package_SO:SOIC-8_3.9x4.9mm_P1.27mm, F.Cu at (121.8, 69.7)
- moved REF** 25.7 mm to (131.2, 83.2)
Routing:
- net +3V3: track 0.00 -> 17.4 mm
- net +5V: track 0.00 -> 11.3 mm
- added copper zone on B.Cu, net GND
- added copper zone on F.Cu, net GND
Other:
- board outline added: 65 x 56.5 mm

Commit message: First finished draft HW
Parts:
- added D3: LED, Diode_SMD:D_1206_3216Metric, F.Cu at (154.5, 74.8)
- added D4: LED, Diode_SMD:D_1206_3216Metric, F.Cu at (160.5, 74.8)
- added D5: LED, Diode_SMD:D_1206_3216Metric, F.Cu at (157.5, 74.8)
- added R5: R_Small, Resistor_SMD:R_0603_1608Metric, F.Cu at (153.2, 68.8)
- added R6: R_Small, Resistor_SMD:R_0603_1608Metric, F.Cu at (153.2, 64.8)
- added R7: R_Small, Resistor_SMD:R_0603_1608Metric, F.Cu at (153.2, 66.8)
- added REF**: MountingHole_3.2mm_M3, MountingHole:MountingHole_3.2mm_M3, F.Cu at (102.2, 59.0)
- added REF**: MountingHole_3.2mm_M3, MountingHole:MountingHole_3.2mm_M3, F.Cu at (160.2, 59.0)
- added REF**: MountingHole_3.2mm_M3, MountingHole:MountingHole_3.2mm_M3, F.Cu at (102.2, 108.0)
- added REF**: KiCad-Logo2_12mm_SilkScreen, Symbol:KiCad-Logo2_12mm_SilkScreen, F.Cu at (121.2, 97.2)
- added REF**: MountingHole_3.2mm_M3, MountingHole:MountingHole_3.2mm_M3, F.Cu at (160.2, 108.0)
- BZ1: footprint Buzzer_Beeper:Buzzer_15x7.5RM7.6 -> Buzzer_Beeper:Buzzer_12x9.5RM7.6
- moved C2 45.2 mm to (111.8, 70.0), turned to 180 degrees
- moved BZ1 42.7 mm to (148.0, 87.8), turned to 90 degrees
- moved R4 31.8 mm to (127.8, 69.0), turned to 270 degrees
- moved R3 31.7 mm to (125.8, 69.0), turned to 270 degrees
- moved D1 30.6 mm to (134.8, 66.0), turned to 270 degrees
- moved Q1 30.3 mm to (148.8, 71.2), turned to 270 degrees
- moved J3 26.5 mm to (108.9, 78.7), turned to 270 degrees
- moved D2 22.5 mm to (130.2, 66.0)
- moved L1 20.0 mm to (116.8, 78.8), turned to 270 degrees
- moved J4 19.8 mm to (137.8, 80.0), turned to 270 degrees
- moved Q2 19.6 mm to (141.8, 71.2), turned to 270 degrees
- moved L2 18.7 mm to (114.8, 78.8), turned to 270 degrees
- moved R1 17.5 mm to (147.8, 65.5), turned to 90 degrees
- moved R2 12.9 mm to (145.2, 65.5), turned to 90 degrees
- moved C3 3.92 mm to (111.8, 71.8), turned to 180 degrees
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Routing:
- net +5V: track 11.3 -> 78.0 mm, vias 0 -> 1
- net Net-(J2-Pad2): track 0.00 -> 51.7 mm, vias 0 -> 2
- net +3V3: track 17.4 -> 65.1 mm, vias 0 -> 2
- net /SO: track 0.00 -> 32.3 mm
- net /SCK: track 0.00 -> 28.0 mm, vias 0 -> 3
- net Net-(D1-Pad2): track 0.00 -> 26.9 mm
- net /CS: track 0.00 -> 26.1 mm
- net Net-(J1-Pad27): track 0.00 -> 17.7 mm, vias 0 -> 2
- net Net-(D2-Pad2): track 0.00 -> 14.7 mm
- net Net-(J1-Pad29): track 0.00 -> 11.7 mm, vias 0 -> 1
- net Net-(J1-Pad31): track 0.00 -> 11.3 mm, vias 0 -> 1
- net Net-(D4-Pad2): track 0.00 -> 11.3 mm
- net Net-(C1-Pad2): track 0.00 -> 10.9 mm, vias 0 -> 2
- net Net-(J3-Pad2): track 0.00 -> 9.61 mm
- net Net-(C1-Pad1): track 0.00 -> 9.03 mm
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
Commit message: HW rev1
Parts:
- removed the REF** at (102.2, 59.0)
- removed the REF** at (160.2, 59.0)
- removed the REF** at (102.2, 108.0)
- removed the REF** at (160.2, 108.0)
- added R8: 1k, Resistor_SMD:R_0603_1608Metric, F.Cu at (148.0, 68.5)
- added R9: 1k, Resistor_SMD:R_0603_1608Metric, F.Cu at (142.2, 68.5)
- added REF**: MountingHole_3mm, MountingHole:MountingHole_3mm, F.Cu at (102.2, 59.0)
- added REF**: MountingHole_3mm, MountingHole:MountingHole_3mm, F.Cu at (160.2, 59.0)
- added REF**: MountingHole_3mm, MountingHole:MountingHole_3mm, F.Cu at (160.2, 108.0)
- added REF**: MountingHole_3mm, MountingHole:MountingHole_3mm, F.Cu at (102.2, 108.0)
- moved REF** 7.10 mm to (119.4, 104.1)
Routing:
- net Net-(Q1-Pad2): track 7.17 -> 7.85 mm
- net GND: vias 56 -> 55
Other:
- board text added: "RPI SMD Oven 1912 - ATHIR"

Commit message: Sorry future me
Changed lines of the file:
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@@
-(kicad_pcb (version 20171130) (host pcbnew "(5.0.0)")
+(kicad_pcb (version 20171130) (host pcbnew "(5.1.0)-1")
   (general
     (thickness 1.6)
@@
     (zone_45_only no)
     (trace_min 0.2)
-    (segment_width 0.2)
-    (edge_width 0.15)
     (via_size 0.8)
     (via_drill 0.4)
@@
     (uvia_min_size 0.2)
     (uvia_min_drill 0.1)
+    (edge_width 0.15)
+    (segment_width 0.2)
     (pcb_text_width 0.3)
     (pcb_text_size 1.5 1.5)
@@
   (gr_arc (start 160.7 57.95) (end 163.7 57.95) (angle -90) (layer Edge.Cuts) (width 0.15))
   (gr_line (start 163.7 108.45) (end 163.7 57.95) (layer Edge.Cuts) (width 0.15))
-  (gr_line (start 160.7 54.95) (end 101.69 54.95) (layer Edge.Cuts) (width 0.15))
+  (gr_line (start 160.7 54.95) (end 101.7 54.95) (layer Edge.Cuts) (width 0.15))
   (segment (start 107.1 57.66) (end 105.75 59.01) (width 0.25) (layer F.Cu) (net 1))
   (segment (start 105.75 59.01) (end 105.75 63.2) (width 0.25) (layer F.Cu) (net 1))
