File: Hardware/rpismdoven/rpismdoven.sch (KiCad schematic (older format))
At the start: 18 parts, among them J1 Raspberry_Pi_2_3, J2 T-PROBE, J3 MAX31855-BREAKOUT, Q1 2N2219, U1 MAX31855TASA

Commit message: bump hw
Parts:
- removed BZ?: Buzzer, symbol Device:Buzzer
- removed FL?: ACP3225, symbol athir:ACP3225
- removed J?: Jack-DC, symbol Connector:Jack-DC
- added J?: Conn_01x02_Female, symbol Connector:Conn_01x02_Female
- added Q?: 2N2219, Package_TO_SOT_THT:TO-39-3, symbol Transistor_BJT:2N2219
- added R? (x2): 10k, symbol Device:R_Small
Connections:
- net labels added: +5V, BUZZ
- net labels removed: +12V
- wire segments 47 -> 53
Other:
- moved on the sheet: Q1
Changed lines of the file:
@@
 L Transistor_BJT:2N2219 Q1
 U 1 1 5C858B83
-P 4225 6600
-F 0 "Q1" H 4416 6646 50  0000 L CNN
-F 1 "2N2219" H 4416 6555 50  0000 L CNN
-F 2 "Package_TO_SOT_THT:TO-39-3" H 4425 6525 50  0001 L CIN
-F 3 "http://www.onsemi.com/pub_link/Collateral/2N2219-D.PDF" H 4225 6600 50  0001 L CNN
-	1    4225 6600
+P 4600 6300
+F 0 "Q1" H 4791 6346 50  0000 L CNN
+F 1 "2N2219" H 4791 6255 50  0000 L CNN
+F 2 "Package_TO_SOT_THT:TO-39-3" H 4800 6225 50  0001 L CIN
+F 3 "http://www.onsemi.com/pub_link/Collateral/2N2219-D.PDF" H 4600 6300 50  0001 L CNN
+	1    4600 6300
 	1    0    0    -1
 $EndComp
-Text Label 4025 6600 2    50   ~ 0
+Text Label 3975 6300 2    50   ~ 0
 PWM
 Text Label 5825 3250 0    50   ~ 0
@@
 $EndComp
 $Comp
-L Connector:Jack-DC J?
-U 1 1 5C87D6BF
-P 7700 4875
-F 0 "J?" H 7755 5200 50  0000 C CNN
-F 1 "Jack-DC" H 7755 5109 50  0000 C CNN
-F 2 "" H 7750 4835 50  0001 C CNN
-F 3 "~" H 7750 4835 50  0001 C CNN
-	1    7700 4875
+L Transistor_BJT:2N2219 Q?
+U 1 1 5C88006E
+P 2525 5525
+F 0 "Q?" H 2716 5571 50  0000 L CNN
+F 1 "2N2219" H 2716 5480 50  0000 L CNN
+F 2 "Package_TO_SOT_THT:TO-39-3" H 2725 5450 50  0001 L CIN
+F 3 "http://www.onsemi.com/pub_link/Collateral/2N2219-D.PDF" H 2525 5525 50  0001 L CNN
+	1    2525 5525
 	1    0    0    -1
 $EndComp
 $Comp
-L athir:ACP3225 FL?
-U 1 1 5C87D79B
-P 8450 4875
-F 0 "FL?" H 8450 5222 60  0000 C CNN
-F 1 "ACP3225" H 8450 5116 60  0000 C CNN
-F 2 "" H 8450 5025 60  0001 C CNN
-F 3 "" H 8450 5025 60  0001 C CNN
-	1    8450 4875
+L power:+5V #PWR?
+U 1 1 5C880836
+P 2650 4700
+F 0 "#PWR?" H 2650 4550 50  0001 C CNN
+F 1 "+5V" H 2665 4873 50  0000 C CNN
+F 2 "" H 2650 4700 50  0001 C CNN
+F 3 "" H 2650 4700 50  0001 C CNN
+	1    2650 4700
+	1    0    0    -1
+$EndComp
+$Comp
+L Device:R_Small R?
+U 1 1 5C880E08
+P 4200 6300
+F 0 "R?" V 4004 6300 50  0000 C CNN
+F 1 "10k" V 4095 6300 50  0000 C CNN
+F 2 "" H 4200 6300 50  0001 C CNN
+F 3 "~" H 4200 6300 50  0001 C CNN
+	1    4200 6300
+	0    1    1    0
+$EndComp
+Wire Wire Line
+	4100 6300 3975 6300
+Wire Wire Line
+	4300 6300 4400 6300
+$Comp
+L Device:R_Small R?
+U 1 1 5C88374F
+P 2100 5525
+F 0 "R?" V 1904 5525 50  0000 C CNN
+F 1 "10k" V 1995 5525 50  0000 C CNN
+F 2 "" H 2100 5525 50  0001 C CNN
+F 3 "~" H 2100 5525 50  0001 C CNN
+	1    2100 5525
+	0    1    1    0
+$EndComp
+Wire Wire Line
+	2200 5525 2325 5525
+Text Label 1950 5525 2    50   ~ 0
+BUZZ
+Wire Wire Line
+	2000 5525 1950 5525
+Wire Wire Line
+	2700 5100 2625 5100
+Wire Wire Line
+	2625 5100 2625 5325
+$Comp
+L Connector:Conn_01x02_Female J?
+U 1 1 5C885BF8
+P 5050 5900
+F 0 "J?" H 5077 5876 50  0000 L CNN
+F 1 "Conn_01x02_Female" H 5077 5785 50  0000 L CNN
+F 2 "" H 5050 5900 50  0001 C CNN
+F 3 "~" H 5050 5900 50  0001 C CNN
+	1    5050 5900
 	1    0    0    -1
 $EndComp
 Wire Wire Line
-	8250 4775 8000 4775
+	2650 4700 2650 4900
 Wire Wire Line
-	8000 4975 8250 4975
+	2650 4900 2700 4900
 $Comp
-L power:+12V #PWR?
-U 1 1 5C87E71F
-P 8800 4725
-F 0 "#PWR?" H 8800 4575 50  0001 C CNN
-F 1 "+12V" H 8815 4898 50  0000 C CNN
-F 2 "" H 8800 4725 50  0001 C CNN
-F 3 "" H 8800 4725 50  0001 C CNN
-	1    8800 4725
+L power:+5V #PWR?
+U 1 1 5C886B71
+P 4700 5825
+F 0 "#PWR?" H 4700 5675 50  0001 C CNN
+F 1 "+5V" H 4715 5998 50  0000 C CNN
+F 2 "" H 4700 5825 50  0001 C CNN
+F 3 "" H 4700 5825 50  0001 C CNN
+	1    4700 5825
 	1    0    0    -1
 $EndComp
 Wire Wire Line
-	8800 4725 8800 4775
+	4850 5900 4700 5900
 Wire Wire Line
-	8800 4775 8650 4775
+	4700 5900 4700 5825
 Wire Wire Line
-	8650 4975 8800 4975
+	4850 6000 4700 6000
 Wire Wire Line
-	8800 4975 8800 5025
-$Comp
-L power:GND #PWR?
-U 1 1 5C87F939
-P 8800 5025
-F 0 "#PWR?" H 8800 4775 50  0001 C CNN
-F 1 "GND" H 8805 4852 50  0000 C CNN
-F 2 "" H 8800 5025 50  0001 C CNN
-F 3 "" H 8800 5025 50  0001 C CNN
-	1    8800 5025
-	1    0    0    -1
-$EndComp
-$Comp
-L Device:Buzzer BZ?
-U 1 1 5C87FB61
-P 5425 6500
-F 0 "BZ?" H 5578 6529 50  0000 L CNN
-F 1 "Buzzer" H 5578 6438 50  0000 L CNN
-F 2 "" V 5400 6600 50  0001 C CNN
-F 3 "~" V 5400 6600 50  0001 C CNN
-	1    5425 6500
-	1    0    0    -1
-$EndComp
+	4700 6000 4700 6100
 $EndSCHEMATC

Commit message: bump HW
Parts:
- C1, C2, C3: footprint (none) -> Capacitor_SMD:C_0603_1608Metric
- J1: footprint (none) -> Connector_PinSocket_2.54mm:PinSocket_2x20_P2.54mm_Vertical
- J2: renamed from J?; footprint (none) -> TerminalBlock:TerminalBlock_bornier-2_P5.08mm
- J3: renamed from J2; footprint (none) -> TerminalBlock:TerminalBlock_bornier-2_P5.08mm
- J4: renamed from J3; footprint (none) -> Connector_PinSocket_2.54mm:PinSocket_1x06_P2.54mm_Vertical
- L1, L2: footprint (none) -> Inductor_SMD:L_0603_1608Metric
- Q1: renamed from Q?; footprint Package_TO_SOT_THT:TO-39-3 -> Package_TO_SOT_THT:TO-92
- Q2: renamed from Q1; footprint Package_TO_SOT_THT:TO-39-3 -> Package_TO_SOT_THT:TO-92
- R1, R2: renamed from R?; value 10k -> 1k; footprint (none) -> Resistor_SMD:R_0603_1608Metric
- R3: renamed from R1; footprint (none) -> Resistor_SMD:R_0603_1608Metric
- R4: renamed from R2; footprint (none) -> Resistor_SMD:R_0603_1608Metric
Connections:
- net +3V3: now also J1.1 (3V3), J1.17 (3V3)
- net +5V: now also J1.2 (5V), J1.4 (5V)
- net BUZZ: now also J1.33 (PWM1/GPIO13)
- net GND: now also J1.14 (GND), J1.20 (GND), J1.25 (GND), J1.30 (GND), J1.34 (GND), J1.39 (GND), J1.6 (GND), J1.9 (GND), Q1.1 (E), Q2.1 (E)
- net PWM: now also J1.32 (PWM0/GPIO12); no longer J1.3 (SDA/GPIO2)
- no-connect marks 1 -> 24

Commit message: First finished draft HW
Parts:
- added D3, D4, D5: LED, Diode_SMD:D_1206_3216Metric, symbol Device:LED
- added R5, R6, R7: R_Small, Resistor_SMD:R_0603_1608Metric, symbol Device:R_Small
- BZ1: footprint (none) -> Buzzer_Beeper:Buzzer_12x9.5RM7.6
Connections:
- net GND: now also D3.1 (K), D4.1 (K), D5.1 (K)
- net at J1.27 (ID_SD/GPIO0): now also R5.2
- net at J1.29 (GCLK1/GPIO5): now also R6.2
- net at J1.31 (GCLK2/GPIO6): now also R7.2
- new net: D3.2 (A), R5.1
- new net: D4.2 (A), R6.1
- new net: D5.2 (A), R7.1
- no-connect marks 24 -> 20
Changed lines of the file:
@@
 	9425 2325 9425 2275
 Wire Wire Line
-	9425 2275 9100 2275
-Connection ~ 9100 2275
-Wire Wire Line
 	9425 2525 9425 2725
 Wire Wire Line
@@
 	9600 2325 9600 2275
 Wire Wire Line
-	9600 2275 9425 2275
-Connection ~ 9425 2275
+	9600 2275 9500 2275
 $Comp
 L Diode:1N4148 D1
@@
 F 0 "BZ1" H 2953 5029 50  0000 L CNN
 F 1 "Buzzer" H 2953 4938 50  0000 L CNN
-F 2 "" V 2775 5100 50  0001 C CNN
+F 2 "Buzzer_Beeper:Buzzer_12x9.5RM7.6" V 2775 5100 50  0001 C CNN
 F 3 "~" V 2775 5100 50  0001 C CNN
 	1    2800 5000
@@
 Text Label 5825 4650 0    50   ~ 0
 BUZZ
-NoConn ~ 5825 3550
-NoConn ~ 5825 3650
-NoConn ~ 5825 3750
 NoConn ~ 5825 3950
 NoConn ~ 5825 4050
@@
 NoConn ~ 5825 3250
 NoConn ~ 5825 3350
-NoConn ~ 5825 2950
 NoConn ~ 5825 3050
 NoConn ~ 4225 2950
@@
 Wire Wire Line
 	4925 5275 4925 5225
+$Comp
+L Device:R_Small R5
+U 1 1 5C8BFEE4
+P 6075 2950
+F 0 "R5" V 5879 2950 50  0000 C CNN
+F 1 "R_Small" V 5970 2950 50  0000 C CNN
+F 2 "Resistor_SMD:R_0603_1608Metric" H 6075 2950 50  0001 C CNN
+F 3 "~" H 6075 2950 50  0001 C CNN
+	1    6075 2950
+	0    1    1    0
+$EndComp
+$Comp
+L Device:R_Small R6
+U 1 1 5C8C251B
+P 6100 3650
+F 0 "R6" V 5904 3650 50  0000 C CNN
+F 1 "R_Small" V 5995 3650 50  0000 C CNN
+F 2 "Resistor_SMD:R_0603_1608Metric" H 6100 3650 50  0001 C CNN
+F 3 "~" H 6100 3650 50  0001 C CNN
+	1    6100 3650
+	0    1    1    0
+$EndComp
+$Comp
+L Device:R_Small R7
+U 1 1 5C8C2557
+P 6100 3750
+F 0 "R7" V 5904 3750 50  0000 C CNN
+F 1 "R_Small" V 5995 3750 50  0000 C CNN
+F 2 "Resistor_SMD:R_0603_1608Metric" H 6100 3750 50  0001 C CNN
+F 3 "~" H 6100 3750 50  0001 C CNN
+	1    6100 3750
+	0    1    1    0
+$EndComp
+Wire Wire Line
+	6000 3750 5825 3750
+Wire Wire Line
+	5825 3650 6000 3650
+$Comp
+L Device:LED D3
+U 1 1 5C8C73ED
+P 6425 2950
+F 0 "D3" H 6417 2695 50  0000 C CNN
+F 1 "LED" H 6417 2786 50  0000 C CNN
+F 2 "Diode_SMD:D_1206_3216Metric" H 6425 2950 50  0001 C CNN
+F 3 "~" H 6425 2950 50  0001 C CNN
+	1    6425 2950
+	-1   0    0    1
+$EndComp
+Wire Wire Line
+	6275 2950 6175 2950
+$Comp
+L Device:LED D4
+U 1 1 5C8C9CD9
+P 6450 3650
+F 0 "D4" H 6442 3395 50  0000 C CNN
+F 1 "LED" H 6442 3486 50  0000 C CNN
+F 2 "Diode_SMD:D_1206_3216Metric" H 6450 3650 50  0001 C CNN
+F 3 "~" H 6450 3650 50  0001 C CNN
+	1    6450 3650
+	-1   0    0    1
+$EndComp
+Wire Wire Line
+	6300 3650 6200 3650
+$Comp
+L Device:LED D5
+U 1 1 5C8CC666
+P 6450 3750
+F 0 "D5" H 6442 3495 50  0000 C CNN
+F 1 "LED" H 6442 3586 50  0000 C CNN
+F 2 "Diode_SMD:D_1206_3216Metric" H 6450 3750 50  0001 C CNN
+F 3 "~" H 6450 3750 50  0001 C CNN
+	1    6450 3750
+	-1   0    0    1
+$EndComp
+$Comp
+L power:GND #PWR0101
+U 1 1 5C8CF0F6
+P 6750 3825
+F 0 "#PWR0101" H 6750 3575 50  0001 C CNN
+F 1 "GND" H 6755 3652 50  0000 C CNN
+F 2 "" H 6750 3825 50  0001 C CNN
+F 3 "" H 6750 3825 50  0001 C CNN
+	1    6750 3825
+	1    0    0    -1
+$EndComp
+Wire Wire Line
+	6750 3825 6750 3750
+Wire Wire Line
+	6750 3750 6600 3750
+Wire Wire Line
+	6600 3650 6750 3650
+Wire Wire Line
+	6750 3650 6750 3750
+Connection ~ 6750 3750
+Connection ~ 6750 3650
+$Comp
+L power:+3V3 #PWR0102
+U 1 1 5C8D7FD6
+P 9500 2175
+F 0 "#PWR0102" H 9500 2025 50  0001 C CNN
+F 1 "+3V3" H 9515 2348 50  0000 C CNN
+F 2 "" H 9500 2175 50  0001 C CNN
+F 3 "" H 9500 2175 50  0001 C CNN
+	1    9500 2175
+	1    0    0    -1
+$EndComp
+Wire Wire Line
+	9500 2175 9500 2275
+Connection ~ 9500 2275
+Wire Wire Line
+	9500 2275 9425 2275
+Wire Wire Line
+	6200 3750 6300 3750
+Wire Wire Line
+	5975 2950 5825 2950
+Wire Wire Line
+	6575 2950 6750 2950
+Wire Wire Line
+	6750 2950 6750 3650
 $EndSCHEMATC

Commit message: HW rev1
Parts:
- added R8, R9: 1k, Resistor_SMD:R_0603_1608Metric, symbol Device:R_Small
Connections:
- net GND: now also R8.1, R9.1
- net at Q2.2 (B), R2.1: now also R9.2
- net at Q1.2 (B), R1.1: now also R8.2
Changed lines of the file:
@@
 	4100 6300 3975 6300
 Wire Wire Line
-	4300 6300 4400 6300
+	4300 6300 4350 6300
 $Comp
 L Device:R_Small R1
@@
 $EndComp
 Wire Wire Line
-	2200 5525 2325 5525
+	2200 5525 2250 5525
 Text Label 1950 5525 2    50   ~ 0
 BUZZ
@@
 L power:GND #PWR04
 U 1 1 5C880CFE
-P 4700 6600
-F 0 "#PWR04" H 4700 6350 50  0001 C CNN
-F 1 "GND" H 4705 6427 50  0000 C CNN
-F 2 "" H 4700 6600 50  0001 C CNN
-F 3 "" H 4700 6600 50  0001 C CNN
-	1    4700 6600
-	1    0    0    -1
-$EndComp
-Wire Wire Line
-	4700 6600 4700 6500
+P 4700 6750
+F 0 "#PWR04" H 4700 6500 50  0001 C CNN
+F 1 "GND" H 4705 6577 50  0000 C CNN
+F 2 "" H 4700 6750 50  0001 C CNN
+F 3 "" H 4700 6750 50  0001 C CNN
+	1    4700 6750
+	1    0    0    -1
+$EndComp
+Wire Wire Line
+	4700 6750 4700 6675
 $Comp
 L power:GND #PWR01
 U 1 1 5C881B9B
-P 2625 5800
-F 0 "#PWR01" H 2625 5550 50  0001 C CNN
-F 1 "GND" H 2630 5627 50  0000 C CNN
-F 2 "" H 2625 5800 50  0001 C CNN
-F 3 "" H 2625 5800 50  0001 C CNN
-	1    2625 5800
-	1    0    0    -1
-$EndComp
-Wire Wire Line
-	2625 5725 2625 5800
+P 2625 5900
+F 0 "#PWR01" H 2625 5650 50  0001 C CNN
+F 1 "GND" H 2630 5727 50  0000 C CNN
+F 2 "" H 2625 5900 50  0001 C CNN
+F 3 "" H 2625 5900 50  0001 C CNN
+	1    2625 5900
+	1    0    0    -1
+$EndComp
+Wire Wire Line
+	2625 5725 2625 5850
 $Comp
 L power:+5V #PWR05
@@
 Wire Wire Line
 	6750 2950 6750 3650
+$Comp
+L Device:R_Small R9
+U 1 1 5C8AD69A
+P 4350 6525
+F 0 "R9" V 4154 6525 50  0000 C CNN
+F 1 "1k" V 4245 6525 50  0000 C CNN
+F 2 "Resistor_SMD:R_0603_1608Metric" H 4350 6525 50  0001 C CNN
+F 3 "~" H 4350 6525 50  0001 C CNN
+	1    4350 6525
+	-1   0    0    1
+$EndComp
+Wire Wire Line
+	4350 6300 4350 6425
+Connection ~ 4350 6300
+Wire Wire Line
+	4350 6300 4400 6300
+Wire Wire Line
+	4350 6625 4350 6675
+Wire Wire Line
+	4350 6675 4700 6675
+Connection ~ 4700 6675
+Wire Wire Line
+	4700 6675 4700 6500
+$Comp
+L Device:R_Small R8
+U 1 1 5C8B6CD4
+P 2250 5675
+F 0 "R8" V 2054 5675 50  0000 C CNN
+F 1 "1k" V 2145 5675 50  0000 C CNN
+F 2 "Resistor_SMD:R_0603_1608Metric" H 2250 5675 50  0001 C CNN
+F 3 "~" H 2250 5675 50  0001 C CNN
+	1    2250 5675
+	-1   0    0    1
+$EndComp
+Wire Wire Line
+	2250 5525 2250 5575
+Connection ~ 2250 5525
+Wire Wire Line
+	2250 5525 2325 5525
+Wire Wire Line
+	2250 5775 2250 5850
+Wire Wire Line
+	2250 5850 2625 5850
+Connection ~ 2625 5850
+Wire Wire Line
+	2625 5850 2625 5900
 $EndSCHEMATC

Commit message: Sorry future me
Parts:
- U1: symbol Sensor_Temperature:MAX31855TASA -> rpismdoven-rescue:MAX31855TASA-Sensor_Temperature
Changed lines of the file:
@@
 EESchema Schematic File Version 4
 LIBS:rpismdoven-cache
-EELAYER 26 0
+EELAYER 30 0
 EELAYER END
 $Descr A4 11693 8268
@@
 $EndComp
 $Comp
-L Sensor_Temperature:MAX31855TASA U1
+L rpismdoven-rescue:MAX31855TASA-Sensor_Temperature U1
 U 1 1 5C862CC5
 P 8450 2925
